File: pcb-mini/epaper-driver.kicad_sch (KiCad schematic)
At the start: 18 parts, among them J15 Conn_01x24, Q3 BSS138

Commit message: [pcb] mini: add/fix LCSC refs
Parts:
- C21, C24, C25, C26, C27, C28: value 1uF/25V -> 1uF; LCSC (none) -> C15849
- C22, C23: value 1uF/10V -> 1uF; LCSC (none) -> C15849
- R21: footprint Resistor_SMD:R_0603_1608Metric -> Resistor_SMD:R_0402_1005Metric; LCSC (none) -> C25744
Other:
- moved on the sheet: C22, C23, C24, C25, C26, C27, C28
