File: pcb-mini/uC.kicad_sch (KiCad schematic)
At the start: 32 parts, among them SW7 SW_Push, U2 RP2350_80QFN, U6 W25Q128JVS, Y2 ABM8-272-T3

Commit message: [pcb] mini: move boot btn, add silkscreen, add con for ESP32 UART
Parts:
- SW7: footprint Button_Switch_SMD:SW_Push_1P1T_NO_Vertical_Wuerth_434133025816 -> Button_Switch_THT:SW_Tactile_SPST_Angled_PTS645Vx31-2LFS
Changed lines of the file:
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@@
 			)
 		)
-		(property "Footprint" "Button_Switch_SMD:SW_Push_1P1T_NO_Vertical_Wuerth_434133025816"
+		(property "Footprint" "Button_Switch_THT:SW_Tactile_SPST_Angled_PTS645Vx31-2LFS"
 			(at 132.08 114.3 0)
 			(effects

Commit message: [pcb] mini: add decoupling caps, improve power path of screen
Parts:
- R1, R3: value 10K -> 4K7; LCSC C25744 -> (none)
Changed lines of the file:
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@@
 			)
 		)
-		(property "Value" "10K"
+		(property "Value" "4K7"
 			(at 267.208 160.782 90)
 			(effects
@@
 			)
 		)
-		(property "Description" "ok LCSC"
-			(at 272.796 166.37 0)
-			(effects
-				(font
-					(size 1.27 1.27)
-				)
-			)
-		)
-		(property "LCSC" "C25744"
+		(property "Description" "LCSC TODO /!\\"
+			(at 273.304 169.926 0)
+			(effects
+				(font
+					(size 1.27 1.27)
+				)
+			)
+		)
+		(property "LCSC" ""
 			(at 269.24 162.56 0)
 			(effects
@@
 			)
 		)
-		(property "Value" "10K"
+		(property "Value" "4K7"
 			(at 274.828 159.512 90)
 			(effects
@@
 			)
 		)
-		(property "LCSC" "C25744"
+		(property "LCSC" ""
 			(at 276.86 161.29 0)
 			(effects
